File: Hardware/Node.sch (EAGLE design)
At the start: 54 parts, among them J1 10118193-0001LF, SW1 FSM4JSMA, U1 WS2813A, U10 WS2813A, U11 WS2813A, U12 WS2813A, U13 ESP-WROOM-02, U14 MIC23050-SYML-TR, U15 74LVC1T45FW4-7, U16 CD74HC4067M96DW24-L, U2 WS2813A, U3 WS2813A, U4 WS2813A, U5 WS2813A, U6 WS2813A, U7 WS2813A, U8 WS2813A, U9 WS2813A

Commit message: Modified Hardware and added eagle libs.
Parts:
- removed C1, C16, C2, C3, C4, C5, C6, C7: 100E-6, rcl:C-EUC0402K
- removed R1, R13, R2, R3, R4, R5, R6, R7: 330, rcl:R-EU_R0402
- removed U10, U11, U12, U9: WS2813A, WS2813A:WS2813A
- added C12, C17, C18, C19: 100E-6, rcl:C-EUC0402K
- added R17, R18, R19, R20, R21, R22, R23, R24: 10E6, rcl:R-EU_R0402
- added R25, R26, R27, R28: 330, rcl:R-EU_R0402
- added SJ10, SJ11, SJ4, SJ5, SJ6, SJ7, SJ8, SJ9: (no value), jumper:SJ2W
Connections:
- net IO0 renamed BOOT0
- net IO15 renamed BOOT2
- net IO2 renamed BOOT1
- net N$46 renamed SENSE1
- net N$47 renamed SENSE2
- net N$48 renamed SENSE3
- net N$49 renamed SENSE4
- net N$50 renamed SENSE5
- net N$51 renamed SENSE6
- net N$52 renamed SENSE7
- net N$53 renamed SENSE8
- removed net D10D11: U10.DIN, U9.DO
- removed net D11D12: U10.DO, U11.BIN, U11.DIN
- removed net D8D9: U7.DO, U8.DIN
- removed net D9D10: U8.DO, U9.DIN
- removed net IO12: U13.IO12
- removed net IO13: U13.IO13
- removed net IO14: U13.IO14
- removed net IO16: U13.IO16
- removed net IO4: U13.IO4
- removed net N$10: R5.2, U5.VCC
- removed net N$11: C5.1, R5.1, U5.VDD
- removed net N$14: R13.2, U12.VCC
- removed net N$15: U1.BIN
- removed net N$16: R6.2, U6.VCC
- removed net N$17: C6.1, R6.1, U6.VDD
- removed net N$18: R7.2, U7.VCC
- removed net N$19: C7.1, R7.1, U7.VDD
- removed net N$2: R1.2, U1.VCC
- removed net N$28: U2.BIN
- removed net N$3: C1.1, R1.1, U1.VDD
- removed net N$4: R2.2, U2.VCC
- removed net N$5: C2.1, R2.1, U2.VDD
- removed net N$54 (its old number): U16A.I8
- removed net N$55 (its old number): U16A.I9
- removed net N$56 (its old number): U16A.I10
- removed net N$58 (its old number): U16A.I12
- removed net N$59 (its old number): U16A.I13
- removed net N$6: R3.2, U3.VCC
- removed net N$60: U16A.I14
- removed net N$61: U16A.I15
- removed net N$62: U16A.COMMONINPUT/OUTPUT
- removed net N$7: C3.1, R3.1, U3.VDD
- removed net N$8: R4.2, U4.VCC
- removed net N$9: C4.1, R4.1, U4.VDD
- new net ADDR0: R20.2, U16A.I8
- new net ADDR1: R21.2, U16A.I9
- new net ADDR2: R22.2, U16A.I10
- new net ADDR3: R23.2, U16A.I11
- new net ADDR4: R17.2, U16A.I12
- new net ADDR5: R18.2, U16A.I13
- new net ADDR6: R19.2, U16A.I14
- new net ADDR7: R24.2, U16A.I15
- new net N$36: C17.1, R26.1, U6.VDD
- new net N$42: R17.1, SJ4.2
- new net N$43: R18.1, SJ5.2
- new net N$44: R19.1, SJ6.2
- new net N$45: R20.1, SJ7.2
- new net N$46: R21.1, SJ8.2
- new net N$47: R22.1, SJ9.2
- new net N$48: R23.1, SJ10.2
- new net N$49: R27.2, U7.VCC
- new net N$50: C18.1, R27.1, U7.VDD
- new net N$51: R28.2, U8.VCC
- new net N$52: C19.1, R28.1, U8.VDD
- net 3V3: now also SJ10.1, SJ11.1, SJ4.1, SJ5.1, SJ6.1, SJ7.1, SJ8.1, SJ9.1
- net 5V: now also C8.1, R8.1, U1.VDD; no longer C16.1, R13.1, U12.VDD
- net ADC_CHANNEL: now also U16A.COMMONINPUT/OUTPUT
- net D1: now also U1.DIN, U2.BIN; no longer U12.DIN
- net D1D2: now also U1.DO, U2.DIN; no longer U1.DIN, U12.DO
- net D2D3: now also U2.DO, U3.DIN; no longer U1.DO, U2.DIN
- net D3D4: now also U3.DO, U4.DIN; no longer U2.DO, U3.DIN
- net D4D5: now also U4.DO, U5.DIN; no longer U3.DO, U4.DIN
- net D5D6: now also U5.DO, U6.DIN; no longer U4.DO, U5.DIN
- net D6D7: now also U6.DO, U7.DIN; no longer U5.DO, U6.DIN
- net D7D8: now also U7.DO, U8.DIN; no longer U6.DO, U7.DIN
- net DOUT: now also U8.DO; no longer U11.DO
- net GND: now also C12.2, C17.2, C18.2, C19.2, SJ10.3, SJ11.3, SJ4.3, SJ5.3, SJ6.3, SJ7.3, SJ8.3, SJ9.3, U1.BIN; no longer C1.2, C16.2, C2.2, C3.2, C4.2, C5.2, C6.2, C7.2, U10.GND, U11.GND, U12.BIN, U12.GND, U9.GND
- net LEDIN3V3: now also U13.IO4
- net N$20: now also U1.VCC; no longer U8.VCC
- net N$21: now also R9.2, U2.VCC; no longer C8.1, R8.1, U8.VDD
- net N$22: now also C9.1, R9.1, U2.VDD; no longer R9.2, U9.VCC
- net N$23: now also R10.2, U3.VCC; no longer C9.1, R9.1, U9.VDD
- net N$24: now also C10.1, R10.1, U3.VDD; no longer R10.2, U10.VCC
- net N$25: now also R11.2, U4.VCC; no longer C10.1, R10.1, U10.VDD
- net N$26: now also C11.1, R11.1, U4.VDD; no longer R11.2, U11.VCC
- net N$27: now also R25.2, U5.VCC; no longer C11.1, R11.1, U11.VDD
- net N$32: now also C12.1, R25.1, U5.VDD; no longer U10.BIN
- net N$33: now also R26.2, U6.VCC; no longer U9.BIN
- net N$57: now also R24.1, SJ11.2; no longer U16A.I11
- net S0: now also U13.IO12
- net S1: now also U13.IO13
- net S2: now also U13.IO14
- net S3: now also U13.IO16
Other:
- note removed: "LED and driver"

Commit message: Modified Node
Parts:
- removed U16: CD74HC4067M96DW24-L, CD74HC4067M96:CD74HC4067M96DW24-L
- added U9: CD4067BPWRPW24-L, CD4067BPWR:CD4067BPWRPW24-L
Connections:
- net N$1 renamed SW
- net N$12 renamed CFF
- new net 9: U14.9
- new net NC: U14.NC
- new net SNS: C14.2, C15.2, L1.2, U14.SNS
- net 3V3: no longer C14.2, C15.2, L1.2, U14.SNS
- net 5V: no longer U16B.VCC
- net ADC_CHANNEL: now also U9.COMMONOUT/IN; no longer U16A.COMMONINPUT/OUTPUT
- net ADDR0: now also U9.CHANNELIN/OUT8; no longer U16A.I8
- net ADDR1: now also U9.CHANNELIN/OUT9; no longer U16A.I9
- net ADDR2: now also U9.CHANNELIN/OUT10; no longer U16A.I10
- net ADDR3: now also U9.CHANNELIN/OUT11; no longer U16A.I11
- net ADDR4: now also U9.CHANNELIN/OUT12; no longer U16A.I12
- net ADDR5: now also U9.CHANNELIN/OUT13; no longer U16A.I13
- net ADDR6: now also U9.CHANNELIN/OUT14; no longer U16A.I14
- net ADDR7: now also U9.CHANNELIN/OUT15; no longer U16A.I15
- net GND: now also U9.INHIBIT, U9.VSS; no longer U16A.!E, U16B.GND
- net S0: now also U9.A; no longer U16A.S0
- net S1: now also U9.B; no longer U16A.S1
- net S2: now also U9.C; no longer U16A.S2
- net S3: now also U9.D; no longer U16A.S3
- net SENSE1: now also U9.CHANNELIN/OUT0; no longer U16A.I0
- net SENSE2: now also U9.CHANNELIN/OUT1; no longer U16A.I1
- net SENSE3: now also U9.CHANNELIN/OUT2; no longer U16A.I2
- net SENSE4: now also U9.CHANNELIN/OUT3; no longer U16A.I3
- net SENSE5: now also U9.CHANNELIN/OUT4; no longer U16A.I4
- net SENSE6: now also U9.CHANNELIN/OUT5; no longer U16A.I5
- net SENSE7: now also U9.CHANNELIN/OUT6; no longer U16A.I6
- net SENSE8: now also U9.CHANNELIN/OUT7; no longer U16A.I7
- net VCC: now also U9.VDD
