File: Hardware/Node.brd (EAGLE design)
At the start: 160 x 103 mm, 54 parts, among them J1 10118193-0001LF, SW1 FSM4JSMA, U1 WS2813A, U10 WS2813A, U11 WS2813A, U12 WS2813A, U13 ESP-WROOM-02, U14 MIC23050-SYML-TR, U15 74LVC1T45FW4-7, U16 CD74HC4067M96DW24-L, U2 WS2813A, U3 WS2813A, U4 WS2813A, U5 WS2813A, U6 WS2813A, U7 WS2813A, U8 WS2813A, U9 WS2813A

Commit message: Modified Hardware and added eagle libs.
Parts:
- removed C1, C16, C2, C3, C4, C5, C6, C7: 100E-6, rcl:C0402K
- removed R1, R13, R2, R3, R4, R5, R6, R7: 330, rcl:R0402
- removed U10, U11, U12, U9: WS2813A, WS2813A:LED_WS2813A
- added C12, C17, C18, C19: 100E-6, rcl:C0402K
- added R17, R18, R19, R20, R21, R22, R23, R24: 10E6, rcl:R0402
- added R25, R26, R27, R28: 330, rcl:R0402
- added SJ10, SJ11, SJ4, SJ5, SJ6, SJ7, SJ8, SJ9: (no value), jumper:SJ_2
- moved R10 70.4 mm to (27.5, 78.3), flipped to the top
- moved R11 70.1 mm to (8.63, 59.4), flipped to the top
- moved C9 69.9 mm to (58.4, 77.3), flipped to the top, turned to 0 degrees
- moved C10 69.8 mm to (31.6, 77.3), flipped to the top, turned to 0 degrees
- moved R9 69.3 mm to (54.4, 78.1), flipped to the top
- moved C11 68.7 mm to (12.6, 58.4), flipped to the top, turned to 0 degrees
- moved C8 68.7 mm to (77.4, 58.4), flipped to the top, turned to 0 degrees
- moved R8 67.0 mm to (73.0, 59.0), flipped to the top
- moved U8 58.2 mm to (77.3, 31.6)
- moved U7 52.6 mm to (58.4, 12.7)
- moved SW1 50.0 mm to (80.2, 45.0), turned to 90 degrees
- moved U6 46.2 mm to (31.6, 12.7)
- moved R12 43.0 mm to (77.5, 36.2)
- moved C14 38.9 mm to (39.4, 10.5), turned to 180 degrees
- moved U5 38.9 mm to (12.7, 31.6)
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Connections:
- net IO0 renamed BOOT0
- net IO15 renamed BOOT2
- net IO2 renamed BOOT1
- net N$46 renamed SENSE1
- net N$47 renamed SENSE2
- net N$48 renamed SENSE3
- net N$49 renamed SENSE4
- net N$50 renamed SENSE5
- net N$51 renamed SENSE6
- net N$52 renamed SENSE7
- net N$53 renamed SENSE8
- removed net D10D11: U10.4, U9.3
- removed net D11D12: U10.3, U11.4, U11.6
- removed net D8D9: U7.3, U8.4
- removed net D9D10: U8.3, U9.4
- removed net IO12: U13.4
- removed net IO13: U13.5
- removed net IO14: U13.3
- removed net IO16: U13.17
- removed net IO4: U13.10
- removed net N$10: R5.2, U5.1
- removed net N$11: C5.1, R5.1, U5.2
- removed net N$14: R13.2, U12.1
- removed net N$15: U1.6
- removed net N$16: R6.2, U6.1
- removed net N$17: C6.1, R6.1, U6.2
- removed net N$18: R7.2, U7.1
- removed net N$19: C7.1, R7.1, U7.2
- removed net N$2: R1.2, U1.1
- removed net N$28: U2.6
- removed net N$3: C1.1, R1.1, U1.2
- removed net N$4: R2.2, U2.1
- removed net N$5: C2.1, R2.1, U2.2
- removed net N$54 (its old number): U16.23
- removed net N$55 (its old number): U16.22
- removed net N$56 (its old number): U16.21
- removed net N$58 (its old number): U16.19
- removed net N$59 (its old number): U16.18
- removed net N$6: R3.2, U3.1
- removed net N$60: U16.17
- removed net N$61: U16.16
- removed net N$62: U16.1
- removed net N$7: C3.1, R3.1, U3.2
- removed net N$8: R4.2, U4.1
- removed net N$9: C4.1, R4.1, U4.2
- new net ADDR0: R20.2, U16.23
- new net ADDR1: R21.2, U16.22
- new net ADDR2: R22.2, U16.21
- new net ADDR3: R23.2, U16.20
- new net ADDR4: R17.2, U16.19
- new net ADDR5: R18.2, U16.18
- new net ADDR6: R19.2, U16.17
- new net ADDR7: R24.2, U16.16
- new net N$36: C17.1, R26.1, U6.2
- new net N$42: R17.1, SJ4.2
- new net N$43: R18.1, SJ5.2
- new net N$44: R19.1, SJ6.2
- new net N$45: R20.1, SJ7.2
- new net N$46: R21.1, SJ8.2
- new net N$47: R22.1, SJ9.2
- new net N$48: R23.1, SJ10.2
- new net N$49: R27.2, U7.1
- new net N$50: C18.1, R27.1, U7.2
- new net N$51: R28.2, U8.1
- new net N$52: C19.1, R28.1, U8.2
- net 3V3: now also SJ10.1, SJ11.1, SJ4.1, SJ5.1, SJ6.1, SJ7.1, SJ8.1, SJ9.1
- net 5V: now also C8.1, R8.1, U1.2; no longer C16.1, R13.1, U12.2
- net ADC_CHANNEL: now also U16.1
- net D1: now also U1.4, U2.6; no longer U12.4
- net D1D2: now also U1.3, U2.4; no longer U1.4, U12.3
- net D2D3: now also U2.3, U3.4; no longer U1.3, U2.4
- net D3D4: now also U3.3, U4.4; no longer U2.3, U3.4
- net D4D5: now also U4.3, U5.4; no longer U3.3, U4.4
- net D5D6: now also U5.3, U6.4; no longer U4.3, U5.4
- net D6D7: now also U6.3, U7.4; no longer U5.3, U6.4
- net D7D8: now also U7.3, U8.4; no longer U6.3, U7.4
- net DOUT: now also U8.3; no longer U11.3
- net GND: now also C12.2, C17.2, C18.2, C19.2, SJ10.3, SJ11.3, SJ4.3, SJ5.3, SJ6.3, SJ7.3, SJ8.3, SJ9.3, U1.6; no longer C1.2, C16.2, C2.2, C3.2, C4.2, C5.2, C6.2, C7.2, U10.5, U11.5, U12.5, U12.6, U9.5
- net LEDIN3V3: now also U13.10
- net N$20: now also U1.1; no longer U8.1
- net N$21: now also R9.2, U2.1; no longer C8.1, R8.1, U8.2
- net N$22: now also C9.1, R9.1, U2.2; no longer R9.2, U9.1
- net N$23: now also R10.2, U3.1; no longer C9.1, R9.1, U9.2
- net N$24: now also C10.1, R10.1, U3.2; no longer R10.2, U10.1
- net N$25: now also R11.2, U4.1; no longer C10.1, R10.1, U10.2
- net N$26: now also C11.1, R11.1, U4.2; no longer R11.2, U11.1
- net N$27: now also R25.2, U5.1; no longer C11.1, R11.1, U11.2
- net N$32: now also C12.1, R25.1, U5.2; no longer U10.6
- net N$33: now also R26.2, U6.1; no longer U9.6
- net N$57: now also R24.1, SJ11.2; no longer U16.20
- net S0: now also U13.4
- net S1: now also U13.5
- net S2: now also U13.3
- net S3: now also U13.17
Routing:
- net N$75: track 180.0 -> 0.00 mm
- net N$76: track 120.0 -> 0.00 mm
- net N$77: track 60.0 -> 0.00 mm
- net N$9: track 0.00 -> 51.4 mm
- net N$8: track 0.00 -> 51.4 mm
- net N$7: track 0.00 -> 51.4 mm
- net N$6: track 0.00 -> 51.4 mm
- net N$5: track 0.00 -> 51.4 mm
- net N$4: track 0.00 -> 51.4 mm
- net N$3: track 0.00 -> 51.4 mm
- net N$10: track 0.00 -> 51.4 mm
- net TX: track 0.00 -> 35.6 mm
- net RX: track 0.00 -> 34.1 mm
- net D3D4: track 0.00 -> 27.0 mm
- net S2: track 0.00 -> 23.0 mm, vias 0 -> 1
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Other:
- outline, holes or cut-outs redrawn

Commit message: Modified Node
Parts:
- removed U16: CD74HC4067M96DW24-L, CD74HC4067M96:DW24-L
- added U9: CD4067BPWRPW24-L, CD4067BPWR:PW24-L
- moved C8 164.2 mm to (-86.4, 71.1), flipped to the bottom
- moved SJ3 149.6 mm to (-88.9, 66.0), turned to 0 degrees
- moved R16 144.5 mm to (-86.4, 57.1)
- moved R28 143.5 mm to (-67.3, 62.2), flipped to the bottom, turned to 0 degrees
- moved C9 138.5 mm to (-80.0, 71.1), flipped to the bottom
- moved R27 135.6 mm to (-72.4, 62.2), flipped to the bottom, turned to 0 degrees
- moved U15 134.8 mm to (-90.2, 74.9), flipped to the bottom
- moved SJ4 131.4 mm to (-82.5, 66.0), flipped to the bottom, turned to 0 degrees
- moved R8 130.2 mm to (-57.1, 62.2), flipped to the bottom, turned to 0 degrees
- moved R17 128.6 mm to (-80.0, 57.1), flipped to the bottom, turned to 0 degrees
- moved SW1 127.5 mm to (-44.5, 17.8), turned to 0 degrees
- moved C19 125.7 mm to (-41.9, 71.1), flipped to the bottom
- moved SJ7 125.2 mm to (-63.5, 66.0), flipped to the bottom, turned to 0 degrees
- moved C13 122.3 mm to (-44.5, 26.7), turned to 0 degrees
- moved C18 121.6 mm to (-48.3, 71.1), flipped to the bottom
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Connections:
- net N$1 renamed SW
- net N$12 renamed CFF
- new net 9: U14.9
- new net NC: U14.3
- new net SNS: C14.2, C15.2, L1.2, U14.4
- net 3V3: no longer C14.2, C15.2, L1.2, U14.4
- net 5V: no longer U16.24
- net ADC_CHANNEL: now also U9.1; no longer U16.1
- net ADDR0: now also U9.23; no longer U16.23
- net ADDR1: now also U9.22; no longer U16.22
- net ADDR2: now also U9.21; no longer U16.21
- net ADDR3: now also U9.20; no longer U16.20
- net ADDR4: now also U9.19; no longer U16.19
- net ADDR5: now also U9.18; no longer U16.18
- net ADDR6: now also U9.17; no longer U16.17
- net ADDR7: now also U9.16; no longer U16.16
- net GND: now also U9.12, U9.15; no longer U16.12, U16.15
- net S0: now also U9.10; no longer U16.10
- net S1: now also U9.11; no longer U16.11
- net S2: now also U9.14; no longer U16.14
- net S3: now also U9.13; no longer U16.13
- net SENSE1: now also U9.9; no longer U16.9
- net SENSE2: now also U9.8; no longer U16.8
- net SENSE3: now also U9.7; no longer U16.7
- net SENSE4: now also U9.6; no longer U16.6
- net SENSE5: now also U9.5; no longer U16.5
- net SENSE6: now also U9.4; no longer U16.4
- net SENSE7: now also U9.3; no longer U16.3
- net SENSE8: now also U9.2; no longer U16.2
- net VCC: now also U9.24
Routing:
- net N$9: track 51.4 -> 0.00 mm
- net N$10: track 51.4 -> 0.00 mm
- net N$3: track 51.4 -> 11.4 mm
- net N$4: track 51.4 -> 11.9 mm
- net N$5: track 51.4 -> 12.4 mm
- net N$6: track 51.4 -> 13.0 mm
- net N$7: track 51.4 -> 13.5 mm
- net N$8: track 51.4 -> 14.0 mm
- net TX: track 35.6 -> 0.00 mm
- net RX: track 34.1 -> 0.00 mm
- net D3D4: track 27.0 -> 0.00 mm
- net S2: track 23.0 -> 0.00 mm, vias 1 -> 0
- net N$45: track 18.2 -> 0.00 mm
- net N$57: track 15.8 -> 0.00 mm
- net N$46: track 14.0 -> 0.00 mm
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Other:
- board size 160 x 103 mm -> 66 x 66 mm

Commit message: Adapted Circuit
Routing:
- net N$8: track 14.0 -> 0.00 mm
- net N$7: track 13.5 -> 0.00 mm
- net N$6: track 13.0 -> 0.00 mm
- net N$5: track 12.4 -> 0.00 mm
- net N$4: track 11.9 -> 0.00 mm
- net N$3: track 11.4 -> 0.00 mm
- net N$2: track 10.9 -> 0.00 mm
Changed lines of the file:
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@@
 <layer number="43" name="vRestrict" color="2" fill="10" visible="yes" active="yes"/>
 <layer number="44" name="Drills" color="7" fill="1" visible="no" active="yes"/>
-<layer number="45" name="Holes" color="7" fill="1" visible="no" active="yes"/>
+<layer number="45" name="Holes" color="7" fill="1" visible="yes" active="yes"/>
 <layer number="46" name="Milling" color="3" fill="1" visible="no" active="yes"/>
 <layer number="47" name="Measures" color="7" fill="1" visible="no" active="yes"/>
@@
 <wire x1="9.906" y1="25.019" x2="4.572" y2="25.019" width="0.0762" layer="20"/>
 <wire x1="4.572" y1="25.019" x2="4.572" y2="19.685" width="0.0762" layer="20"/>
+<hole x="29.718" y="63.881" drill="0.35"/>
+<hole x="36.322" y="63.881" drill="0.35"/>
+<rectangle x1="25.019" y1="8.255" x2="25.527" y2="9.398" layer="16"/>
+<rectangle x1="25.019" y1="6.604" x2="25.527" y2="7.747" layer="16"/>
+<rectangle x1="25.019" y1="5.08" x2="25.527" y2="6.223" layer="16"/>
+<rectangle x1="19.05" y1="8.255" x2="19.685" y2="9.398" layer="16"/>
+<rectangle x1="19.05" y1="6.731" x2="19.685" y2="7.747" layer="16"/>
+<rectangle x1="19.05" y1="5.08" x2="19.685" y2="6.223" layer="16"/>
+<rectangle x1="9.906" y1="20.193" x2="10.414" y2="21.209" layer="16"/>
+<rectangle x1="9.906" y1="21.844" x2="10.414" y2="22.86" layer="16"/>
+<rectangle x1="9.906" y1="23.368" x2="10.414" y2="24.511" layer="16"/>
+<rectangle x1="3.937" y1="23.368" x2="4.572" y2="24.511" layer="16"/>
+<rectangle x1="3.937" y1="21.717" x2="4.572" y2="22.86" layer="16"/>
+<rectangle x1="3.937" y1="20.193" x2="4.572" y2="21.336" layer="16"/>
+<rectangle x1="3.937" y1="44.831" x2="4.572" y2="45.847" layer="16"/>
+<rectangle x1="3.937" y1="43.18" x2="4.572" y2="44.196" layer="16"/>
+<rectangle x1="3.937" y1="41.529" x2="4.572" y2="42.672" layer="16"/>
+<rectangle x1="9.906" y1="41.529" x2="10.414" y2="42.672" layer="16"/>
+<rectangle x1="9.906" y1="43.18" x2="10.414" y2="44.323" layer="16"/>
+<rectangle x1="9.906" y1="44.704" x2="10.414" y2="45.847" layer="16"/>
+<rectangle x1="19.05" y1="59.817" x2="19.685" y2="60.96" layer="16"/>
+<rectangle x1="19.05" y1="58.293" x2="19.685" y2="59.309" layer="16"/>
+<rectangle x1="19.05" y1="56.642" x2="19.685" y2="57.785" layer="16"/>
+<rectangle x1="25.019" y1="56.769" x2="25.527" y2="57.658" layer="16"/>
+<rectangle x1="25.019" y1="58.293" x2="25.527" y2="59.309" layer="16"/>
+<rectangle x1="25.019" y1="59.944" x2="25.527" y2="60.96" layer="16"/>
+<rectangle x1="40.513" y1="59.944" x2="41.021" y2="60.96" layer="16"/>
+<rectangle x1="40.513" y1="56.642" x2="41.021" y2="57.785" layer="16"/>
+<rectangle x1="46.355" y1="56.642" x2="46.99" y2="57.785" layer="16"/>
+<rectangle x1="46.355" y1="58.293" x2="46.99" y2="59.436" layer="16"/>
+<rectangle x1="46.355" y1="59.944" x2="46.99" y2="60.96" layer="16"/>
+<rectangle x1="61.468" y1="44.831" x2="62.103" y2="45.847" layer="16"/>
+<rectangle x1="61.468" y1="43.053" x2="62.103" y2="44.323" layer="16"/>
+<rectangle x1="61.468" y1="41.529" x2="62.103" y2="42.672" layer="16"/>
+<rectangle x1="55.626" y1="41.656" x2="56.134" y2="42.672" layer="16"/>
+<rectangle x1="55.626" y1="43.18" x2="56.134" y2="44.196" layer="16"/>
+<rectangle x1="55.626" y1="44.831" x2="56.134" y2="45.847" layer="16"/>
+<rectangle x1="55.626" y1="23.368" x2="56.134" y2="24.511" layer="16"/>
+<rectangle x1="55.626" y1="21.844" x2="56.134" y2="22.86" layer="16"/>
+<rectangle x1="55.626" y1="20.193" x2="56.134" y2="21.209" layer="16"/>
+<rectangle x1="61.468" y1="20.193" x2="62.103" y2="21.336" layer="16"/>
+<rectangle x1="61.468" y1="21.717" x2="62.103" y2="22.86" layer="16"/>
+<rectangle x1="61.468" y1="23.368" x2="62.103" y2="24.511" layer="16"/>
+<rectangle x1="40.513" y1="8.255" x2="41.021" y2="9.398" layer="16"/>
+<rectangle x1="40.513" y1="6.604" x2="41.021" y2="7.747" layer="16"/>
+<rectangle x1="40.513" y1="5.08" x2="41.021" y2="6.096" layer="16"/>
+<rectangle x1="46.355" y1="5.08" x2="46.99" y2="6.096" layer="16"/>
+<rectangle x1="46.355" y1="6.604" x2="46.99" y2="7.747" layer="16"/>
+<rectangle x1="46.355" y1="8.255" x2="46.99" y2="9.398" layer="16"/>
 </plain>
 <attributes>
@@
 <contactref element="U8" pad="3"/>
 </signal>
-<signal name="N$2">
-<wire x1="25.146" y1="9.906" x2="25.146" y2="4.445" width="0.1524" layer="1"/>
-<wire x1="25.146" y1="4.445" x2="19.685" y2="4.445" width="0.1524" layer="1"/>
-</signal>
-<signal name="N$3">
-<wire x1="19.558" y1="4.318" x2="25.273" y2="4.318" width="0.1524" layer="1"/>
-<wire x1="25.273" y1="4.318" x2="25.273" y2="10.033" width="0.1524" layer="1"/>
-</signal>
-<signal name="N$4">
-<wire x1="25.4" y1="10.16" x2="25.4" y2="4.191" width="0.1524" layer="1"/>
-<wire x1="25.4" y1="4.191" x2="19.431" y2="4.191" width="0.1524" layer="1"/>
-</signal>
-<signal name="N$5">
-<wire x1="19.304" y1="4.064" x2="25.527" y2="4.064" width="0.1524" layer="1"/>
-<wire x1="25.527" y1="4.064" x2="25.527" y2="10.287" width="0.1524" layer="1"/>
-</signal>
-<signal name="N$6">
-<wire x1="25.654" y1="10.414" x2="25.654" y2="3.937" width="0.1524" layer="1"/>
-<wire x1="25.654" y1="3.937" x2="19.177" y2="3.937" width="0.1524" layer="1"/>
-</signal>
-<signal name="N$7">
-<wire x1="19.05" y1="3.81" x2="25.781" y2="3.81" width="0.1524" layer="1"/>
-<wire x1="25.781" y1="3.81" x2="25.781" y2="10.541" width="0.1524" layer="1"/>
-</signal>
-<signal name="N$8">
-<wire x1="25.908" y1="10.668" x2="25.908" y2="3.683" width="0.1524" layer="1"/>
-<wire x1="25.908" y1="3.683" x2="18.923" y2="3.683" width="0.1524" layer="1"/>
-</signal>
 <signal name="NC">
